Commit message: changed to laser_link to laser

File: src/four_wheels_robot/urdf/model.urdf.xacro (robot description, xacro)
@@ -77,12 +77,13 @@
     <xacro:wheel_joint prefix="back_right"  x="-0.12" y="-0.12" r="0"/>
     <!--Adding a lidar-->
-    <link name="laser_link">
+<!-- Adding a LiDAR -->
+    <link name="laser">
         <visual>
             <geometry>
                 <cylinder radius="0.05" length="0.02"/>
             </geometry>
-                <material name="">
-                    <color rgba="0.78 0.55 0.34 1.0"/>
-                </material>
+            <material name="laser_material">
+                <color rgba="0.78 0.55 0.34 1.0"/>
+            </material>
         </visual>
     </link>
@@ -90,6 +91,5 @@
         <origin xyz="0.0 0.0 0.05" rpy="0.0 0.0 0.0"/>
         <parent link="base_link"/>
-        <child link="laser_link"/>
-        <axis xyz="0.0 0.0 0.0"/>
+        <child link="laser"/>
     </joint>
     <!-- Adding IMU SENSOR-->

Commit message: changed wheel radius to 0.045m

File: src/four_wheels_robot/urdf/model.urdf.xacro (robot description, xacro)
@@ -1,5 +1,5 @@
 <?xml version="1.1"?>
 <robot xmlns:xacro="http://ros.org/wiki/xacro" name="four_wheels_robot">
-    <xacro:property name="wheel_radius" value="0.090"/>
+    <xacro:property name="wheel_radius" value="0.045"/>
     <xacro:property name="wheel_length" value="0.04"/>
     <!-- Include control definitions -->

Commit message: changed wheel radius to 0.045m

File: src/four_wheels_robot/urdf/model.urdf.xacro (robot description, xacro)
@@ -1,5 +1,5 @@
 <?xml version="1.1"?>
 <robot xmlns:xacro="http://ros.org/wiki/xacro" name="four_wheels_robot">
-    <xacro:property name="wheel_radius" value="0.045"/>
+    <xacro:property name="wheel_radius" value="0.090"/>
     <xacro:property name="wheel_length" value="0.04"/>
     <!-- Include control definitions -->

Commit message: I have added Btrees maps

File: src/four_wheels_robot/urdf/model.urdf.xacro (robot description, xacro)
@@ -1,6 +1,6 @@
 <?xml version="1.1"?>
 <robot xmlns:xacro="http://ros.org/wiki/xacro" name="four_wheels_robot">
-    <xacro:property name="wheel_radius" value="0.090"/>
-    <xacro:property name="wheel_length" value="0.04"/>
+    <xacro:property name="wheel_radius" value="0.0425"/>
+    <xacro:property name="wheel_length" value="0.02"/>
     <!-- Include control definitions -->
     <!-- <xacro:include filename="$(find four_wheels_robot)/urdf/ros2_wheel_controllers.xacro"/> -->
@@ -43,5 +43,5 @@
             <origin xyz="0.0 0.0 0.0" rpy="0.0 0.0 0.0"/>
             <geometry>
-                <box size="0.5 0.18 0.1"/>
+                <box size="0.3 0.3 0.1"/>
             </geometry>
             <material name="">
@@ -52,5 +52,5 @@
             <origin xyz="0.0 0.0 0.0" rpy="0.0 0.0 0.0"/>
             <geometry>
-                <box size="0.5 0.18 0.1"/>
+                <box size="0.3 0.3 0.1"/>
             </geometry>
         </collision>
@@ -72,8 +72,8 @@
         </joint>
     </xacro:macro>
-    <xacro:wheel_joint prefix="front_left"  x="0.12" y="0.12" r="0"/>
-    <xacro:wheel_joint prefix="front_right" x="0.12" y="-0.12" r="0"/>
-    <xacro:wheel_joint prefix="back_left"   x="-0.12" y="0.12" r="0"/>
-    <xacro:wheel_joint prefix="back_right"  x="-0.12" y="-0.12" r="0"/>
+    <xacro:wheel_joint prefix="front_left"  x="0.10" y="0.162" r="0"/>
+    <xacro:wheel_joint prefix="front_right" x="0.10" y="-0.162" r="0"/>
+    <xacro:wheel_joint prefix="back_left"   x="-0.10" y="0.162" r="0"/>
+    <xacro:wheel_joint prefix="back_right"  x="-0.10" y="-0.162" r="0"/>
     <!--Adding a lidar-->
     <link name="laser_link">
@@ -135,5 +135,5 @@
     <parent link="base_link"/>
     <child link="camera_link"/>
-    <origin xyz="0.25 0.0 0.03" rpy="0 0 0"/>
+    <origin xyz="0.15 0.0 0.03" rpy="0 0 0"/>
  </joint>
 </robot>

Commit message: kol is kool

File: src/four_wheels_robot/urdf/model.urdf.xacro (robot description, xacro)
@@ -1,6 +1,6 @@
 <?xml version="1.1"?>
 <robot xmlns:xacro="http://ros.org/wiki/xacro" name="four_wheels_robot">
-    <xacro:property name="wheel_radius" value="0.090"/>
-    <xacro:property name="wheel_length" value="0.04"/>
+    <xacro:property name="wheel_radius" value="0.0425"/>
+    <xacro:property name="wheel_length" value="0.02"/>
     <!-- Include control definitions -->
     <xacro:include filename="$(find four_wheels_robot)/urdf/ros2_wheel_controllers.xacro"/>
@@ -43,5 +43,5 @@
             <origin xyz="0.0 0.0 0.0" rpy="0.0 0.0 0.0"/>
             <geometry>
-                <box size="0.5 0.18 0.1"/>
+                <box size="0.3 0.3 0.1"/>
             </geometry>
             <material name="">
@@ -52,5 +52,5 @@
             <origin xyz="0.0 0.0 0.0" rpy="0.0 0.0 0.0"/>
             <geometry>
-                <box size="0.5 0.18 0.1"/>
+                <box size="0.3 0.3 0.1"/>
             </geometry>
         </collision>
@@ -72,18 +72,17 @@
         </joint>
     </xacro:macro>
-    <!-- <xacro:wheel_joint prefix="front_left"  x="0.12" y="0.12" r="0"/> -->
-    <!-- <xacro:wheel_joint prefix="front_right" x="0.12" y="-0.12" r="0"/> -->
-    <xacro:wheel_joint prefix="back_left"   x="-0.12" y="0.12" r="0"/>
-    <xacro:wheel_joint prefix="back_right"  x="-0.12" y="-0.12" r="0"/>
+    <!-- <xacro:wheel_joint prefix="front_left"  x="0.10" y="0.162" r="0"/> -->
+    <!-- <xacro:wheel_joint prefix="front_right" x="0.10" y="-0.162" r="0"/> -->
+    <xacro:wheel_joint prefix="back_left"   x="-0.10" y="0.162" r="0"/>
+    <xacro:wheel_joint prefix="back_right"  x="-0.10" y="-0.162" r="0"/>
     <!--Adding a lidar-->
-<!-- Adding a LiDAR -->
-    <link name="laser">
+    <link name="laser_link">
         <visual>
             <geometry>
                 <cylinder radius="0.05" length="0.02"/>
             </geometry>
-            <material name="laser_material">
-                <color rgba="0.78 0.55 0.34 1.0"/>
-            </material>
+                <material name="">
+                    <color rgba="0.78 0.55 0.34 1.0"/>
+                </material>
         </visual>
     </link>
@@ -91,5 +90,6 @@
         <origin xyz="0.0 0.0 0.05" rpy="0.0 0.0 0.0"/>
         <parent link="base_link"/>
-        <child link="laser"/>
+        <child link="laser_link"/>
+        <axis xyz="0.0 0.0 0.0"/>
     </joint>
     <!-- Adding IMU SENSOR-->
@@ -135,5 +135,5 @@
     <parent link="base_link"/>
     <child link="camera_link"/>
-    <origin xyz="0.25 0.0 0.03" rpy="0 0 0"/>
+    <origin xyz="0.15 0.0 0.03" rpy="0 0 0"/>
  </joint>
 </robot>

Commit message: added bt

File: src/four_wheels_robot/urdf/model.urdf.xacro (robot description, xacro)
@@ -43,5 +43,5 @@
             <origin xyz="0.0 0.0 0.0" rpy="0.0 0.0 0.0"/>
             <geometry>
-                <box size="0.3 0.3 0.1"/>
+                <box size="0.3 0.25 0.1"/>
             </geometry>
             <material name="">
@@ -77,5 +77,5 @@
     <xacro:wheel_joint prefix="back_right"  x="-0.10" y="-0.162" r="0"/>
     <!--Adding a lidar-->
-    <link name="laser_link">
+    <link name="laser">
         <visual>
             <geometry>
@@ -88,8 +88,8 @@
     </link>
     <joint name="laser_joint" type="fixed">
-        <origin xyz="0.0 0.0 0.05" rpy="0.0 0.0 0.0"/>
+        <origin xyz="0.0 0.0 0.05" rpy="0.0 0.0 3.142"/>
         <parent link="base_link"/>
-        <child link="laser_link"/>
-        <axis xyz="0.0 0.0 0.0"/>
+        <child link="laser"/>
+        <axis xyz="0.04 0.0 0.0"/>
     </joint>
     <!-- Adding IMU SENSOR-->
